File: PCB design/AM_modulator/_autosave-Mixer.kicad_sch (KiCad schematic)
At the start: 8 parts

Commit message: Placa terminada
Parts:
- gave numbers to parts that had none: 1
Changed lines of the file:
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@@
   (symbol (lib_id "SMA_T:SMA_CONNECTOR") (at 155.702 84.836 0) (unit 1)
     (in_bom yes) (on_board yes)
-    (property "Reference" "J?" (id 0) (at 162.052 84.328 0))
+    (property "Reference" "J4" (id 0) (at 162.052 84.328 0))
     (property "Value" "SMA_CONNECTOR" (id 1) (at 168.91 86.868 0))
     (property "Footprint" "LPRS_SMA_CONNECTOR" (id 2) (at 155.702 84.836 0)
