File: PCB design/AM_modulator/Antenna.kicad_sch (KiCad schematic)
At the start: 4 parts, among them J2 Conn_01x02_Female

Commit message: Nothing useful
Parts:
- Cpi1, Cpi2: footprint (none) -> Capacitor_SMD:C_0805_2012Metric_Pad1.18x1.45mm_HandSolder
Changed lines of the file:
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@@
       (effects (font (size 1.27 1.27)) (justify left))
     )
-    (property "Footprint" "" (id 2) (at 130.2512 84.074 0)
+    (property "Footprint" "Capacitor_SMD:C_0805_2012Metric_Pad1.18x1.45mm_HandSolder" (id 2) (at 130.2512 84.074 0)
       (effects (font (size 1.27 1.27)) hide)
     )
@@
       (effects (font (size 1.27 1.27)) (justify left))
     )
-    (property "Footprint" "" (id 2) (at 110.1852 83.82 0)
+    (property "Footprint" "Capacitor_SMD:C_0805_2012Metric_Pad1.18x1.45mm_HandSolder" (id 2) (at 110.1852 83.82 0)
       (effects (font (size 1.27 1.27)) hide)
     )

Commit message: Avances placa
Parts:
- removed J2: Conn_01x02_Female, Connector_PinSocket_2.54mm:PinSocket_1x02_P2.54mm_Vertical, symbol Connector:Conn_01x02_Female
- added Antena+1, Antena-1: Conn_01x01_Female, Connector_Pin:Pin_D1.4mm_L8.5mm_W2.8mm_FlatFork, symbol Connector:Conn_01x01_Female
- added Cpi11, Cpi21: C, Capacitor_SMD:C_0805_2012Metric_Pad1.18x1.45mm_HandSolder, symbol Device:C
- Lpi1: footprint (none) -> Inductor_THT:L_Toroid_Vertical_L21.6mm_W9.1mm_P8.40mm_Bourns_5700
Connections:
- net GND: now also Lpi1.2, Antena-1.1 (Pin_1), Cpi11.1; no longer Cpi2.2
- net RF_Antenna: now also Cpi2.1, Cpi11.2, Cpi21.1; no longer Lpi1.1
- new net: Antena+1.1 (Pin_1), Cpi2.2, Cpi21.2, Lpi1.1
Other:
- moved on the sheet: Cpi2, Lpi1
Changed lines of the file:
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@@
   (junction (at 129.286 73.66) (diameter 0) (color 0 0 0 0)
   )
+  (junction (at 102.87 73.66) (diameter 0) (color 0 0 0 0)
+  )
   (junction (at 109.22 73.66) (diameter 0) (color 0 0 0 0)
   )
-  (wire (pts (xy 109.22 73.66) (xy 116.332 73.66))
-    (stroke (width 0) (type default) (color 0 0 0 0))
-  )
-  (wire (pts (xy 146.558 76.2) (xy 146.558 78.232))
+  (wire (pts (xy 146.304 82.296) (xy 146.304 84.328))
+    (stroke (width 0) (type default) (color 0 0 0 0))
+  )
+  (wire (pts (xy 102.87 83.82) (xy 102.87 85.344))
     (stroke (width 0) (type default) (color 0 0 0 0))
   )
@@
     (stroke (width 0) (type default) (color 0 0 0 0))
   )
-  (wire (pts (xy 123.952 73.66) (xy 129.286 73.66))
+  (wire (pts (xy 109.22 73.66) (xy 115.062 73.66))
+    (stroke (width 0) (type default) (color 0 0 0 0))
+  )
+  (wire (pts (xy 122.682 73.66) (xy 129.286 73.66))
     (stroke (width 0) (type default) (color 0 0 0 0))
   )
@@
     (stroke (width 0) (type default) (color 0 0 0 0))
   )
-  (wire (pts (xy 98.552 73.66) (xy 109.22 73.66))
+  (wire (pts (xy 102.87 73.66) (xy 102.87 76.2))
+    (stroke (width 0) (type default) (color 0 0 0 0))
+  )
+  (wire (pts (xy 102.87 73.66) (xy 109.22 73.66))
+    (stroke (width 0) (type default) (color 0 0 0 0))
+  )
+  (wire (pts (xy 98.552 73.66) (xy 102.87 73.66))
+    (stroke (width 0) (type default) (color 0 0 0 0))
+  )
+  (wire (pts (xy 129.286 62.484) (xy 129.286 73.66))
+    (stroke (width 0) (type default) (color 0 0 0 0))
+  )
+  (wire (pts (xy 109.22 73.66) (xy 109.22 62.484))
+    (stroke (width 0) (type default) (color 0 0 0 0))
+  )
+  (wire (pts (xy 109.22 62.484) (xy 115.062 62.484))
     (stroke (width 0) (type default) (color 0 0 0 0))
   )
@@
   )
   (wire (pts (xy 129.286 73.66) (xy 146.558 73.66))
+    (stroke (width 0) (type default) (color 0 0 0 0))
+  )
+  (wire (pts (xy 122.682 62.484) (xy 129.286 62.484))
     (stroke (width 0) (type default) (color 0 0 0 0))
   )
@@
     (effects (font (size 1.27 1.27)) (justify right))
   )
+  (symbol (lib_id "Connector:Conn_01x01_Female") (at 151.384 82.296 0) (unit 1)
+    (in_bom yes) (on_board yes) (fields_autoplaced)
+    (property "Reference" "Antena-1" (id 0) (at 152.4 81.0259 0)
+      (effects (font (size 1.27 1.27)) (justify left))
+    )
+    (property "Value" "Conn_01x01_Female" (id 1) (at 152.4 83.5659 0)
+      (effects (font (size 1.27 1.27)) (justify left))
+    )
+    (property "Footprint" "Connector_Pin:Pin_D1.4mm_L8.5mm_W2.8mm_FlatFork" (id 2) (at 151.384 82.296 0)
+      (effects (font (size 1.27 1.27)) hide)
+    )
+    (property "Datasheet" "~" (id 3) (at 151.384 82.296 0)
+      (effects (font (size 1.27 1.27)) hide)
+    )
+    (pin "1")
+  )
+  (symbol (lib_id "power:GND") (at 102.87 85.344 0) (unit 1)
+    (in_bom yes) (on_board yes) (fields_autoplaced)
+    (property "Reference" "#PWR?" (id 0) (at 102.87 91.694 0)
+      (effects (font (size 1.27 1.27)) hide)
+    )
+    (property "Value" "GND" (id 1) (at 102.87 90.17 0))
+    (property "Footprint" "" (id 2) (at 102.87 85.344 0)
+      (effects (font (size 1.27 1.27)) hide)
+    )
+    (property "Datasheet" "" (id 3) (at 102.87 85.344 0)
+      (effects (font (size 1.27 1.27)) hide)
+    )
+    (pin "1")
+  )
   (symbol (lib_id "power:GND") (at 109.22 85.344 0) (unit 1)
     (in_bom yes) (on_board yes) (fields_autoplaced)
@@
     (pin "1")
   )
-  (symbol (lib_id "Device:L") (at 120.142 73.66 90) (unit 1)
-    (in_bom yes) (on_board yes) (fields_autoplaced)
-    (property "Reference" "Lpi1" (id 0) (at 120.142 67.31 90))
-    (property "Value" "L" (id 1) (at 120.142 69.85 90))
-    (property "Footprint" "" (id 2) (at 120.142 73.66 0)
-      (effects (font (size 1.27 1.27)) hide)
-    )
-    (property "Datasheet" "~" (id 3) (at 120.142 73.66 0)
-      (effects (font (size 1.27 1.27)) hide)
-    )
-    (pin "1")
-    (pin "2")
-  )
-  (symbol (lib_id "Device:C") (at 129.286 80.264 0) (unit 1)
-    (in_bom yes) (on_board yes) (fields_autoplaced)
-    (property "Reference" "Cpi2" (id 0) (at 133.35 78.9939 0)
-      (effects (font (size 1.27 1.27)) (justify left))
-    )
-    (property "Value" "C" (id 1) (at 133.35 81.5339 0)
-      (effects (font (size 1.27 1.27)) (justify left))
-    )
-    (property "Footprint" "Capacitor_SMD:C_0805_2012Metric_Pad1.18x1.45mm_HandSolder" (id 2) (at 130.2512 84.074 0)
+  (symbol (lib_id "Device:L") (at 129.286 80.264 0) (unit 1)
+    (in_bom yes) (on_board yes) (fields_autoplaced)
+    (property "Reference" "Lpi1" (id 0) (at 131.572 78.9939 0)
+      (effects (font (size 1.27 1.27)) (justify left))
+    )
+    (property "Value" "L" (id 1) (at 131.572 81.5339 0)
+      (effects (font (size 1.27 1.27)) (justify left))
+    )
+    (property "Footprint" "Inductor_THT:L_Toroid_Vertical_L21.6mm_W9.1mm_P8.40mm_Bourns_5700" (id 2) (at 129.286 80.264 0)
       (effects (font (size 1.27 1.27)) hide)
     )
@@
     (pin "2")
   )
+  (symbol (lib_id "Connector:Conn_01x01_Female") (at 151.638 73.66 0) (unit 1)
+    (in_bom yes) (on_board yes) (fields_autoplaced)
+    (property "Reference" "Antena+1" (id 0) (at 152.4 72.3899 0)
+      (effects (font (size 1.27 1.27)) (justify left))
+    )
+    (property "Value" "Conn_01x01_Female" (id 1) (at 152.4 74.9299 0)
+      (effects (font (size 1.27 1.27)) (justify left))
+    )
+    (property "Footprint" "Connector_Pin:Pin_D1.4mm_L8.5mm_W2.8mm_FlatFork" (id 2) (at 151.638 73.66 0)
+      (effects (font (size 1.27 1.27)) hide)
+    )
+    (property "Datasheet" "~" (id 3) (at 151.638 73.66 0)
+      (effects (font (size 1.27 1.27)) hide)
+    )
+    (pin "1")
+  )
+  (symbol (lib_id "Device:C") (at 118.872 73.66 90) (unit 1)
+    (in_bom yes) (on_board yes) (fields_autoplaced)
+    (property "Reference" "Cpi2" (id 0) (at 118.872 66.294 90))
+    (property "Value" "C" (id 1) (at 118.872 68.834 90))
+    (property "Footprint" "Capacitor_SMD:C_0805_2012Metric_Pad1.18x1.45mm_HandSolder" (id 2) (at 122.682 72.6948 0)
+      (effects (font (size 1.27 1.27)) hide)
+    )
+    (property "Datasheet" "~" (id 3) (at 118.872 73.66 0)
+      (effects (font (size 1.27 1.27)) hide)
+    )
+    (pin "1")
+    (pin "2")
+  )
+  (symbol (lib_id "Device:C") (at 102.87 80.01 180) (unit 1)
+    (in_bom yes) (on_board yes)
+    (property "Reference" "Cpi11" (id 0) (at 96.52 78.486 0)
+      (effects (font (size 1.27 1.27)) (justify right))
+    )
+    (property "Value" "C" (id 1) (at 96.52 81.026 0)
+      (effects (font (size 1.27 1.27)) (justify right))
+    )
+    (property "Footprint" "Capacitor_SMD:C_0805_2012Metric_Pad1.18x1.45mm_HandSolder" (id 2) (at 101.9048 76.2 0)
+      (effects (font (size 1.27 1.27)) hide)
+    )
+    (property "Datasheet" "~" (id 3) (at 102.87 80.01 0)
+      (effects (font (size 1.27 1.27)) hide)
+    )
+    (pin "1")
+    (pin "2")
+  )
   (symbol (lib_id "Device:C") (at 109.22 80.01 0) (unit 1)
     (in_bom yes) (on_board yes) (fields_autoplaced)
@@
     (pin "2")
   )
-  (symbol (lib_id "Connector:Conn_01x02_Female") (at 151.638 73.66 0) (unit 1)
-    (in_bom yes) (on_board yes) (fields_autoplaced)
-    (property "Reference" "J2" (id 0) (at 152.4 73.6599 0)
-      (effects (font (size 1.27 1.27)) (justify left))
-    )
-    (property "Value" "Conn_01x02_Female" (id 1) (at 152.4 76.1999 0)
-      (effects (font (size 1.27 1.27)) (justify left))
-    )
-    (property "Footprint" "Connector_PinSocket_2.54mm:PinSocket_1x02_P2.54mm_Vertical" (id 2) (at 151.638 73.66 0)
-      (effects (font (size 1.27 1.27)) hide)
-    )
-    (property "Datasheet" "~" (id 3) (at 151.638 73.66 0)
-      (effects (font (size 1.27 1.27)) hide)
-    )
-    (pin "1")
-    (pin "2")
-  )
-  (symbol (lib_id "power:GND") (at 146.558 78.232 0) (unit 1)
-    (in_bom yes) (on_board yes) (fields_autoplaced)
-    (property "Reference" "#PWR0113" (id 0) (at 146.558 84.582 0)
-      (effects (font (size 1.27 1.27)) hide)
-    )
-    (property "Value" "GND" (id 1) (at 146.558 83.058 0))
-    (property "Footprint" "" (id 2) (at 146.558 78.232 0)
-      (effects (font (size 1.27 1.27)) hide)
-    )
-    (property "Datasheet" "" (id 3) (at 146.558 78.232 0)
-      (effects (font (size 1.27 1.27)) hide)
-    )
-    (pin "1")
+  (symbol (lib_id "power:GND") (at 146.304 84.328 0) (unit 1)
+    (in_bom yes) (on_board yes) (fields_autoplaced)
+    (property "Reference" "#PWR0113" (id 0) (at 146.304 90.678 0)
+      (effects (font (size 1.27 1.27)) hide)
+    )
+    (property "Value" "GND" (id 1) (at 146.304 89.154 0))
+    (property "Footprint" "" (id 2) (at 146.304 84.328 0)
+      (effects (font (size 1.27 1.27)) hide)
+    )
+    (property "Datasheet" "" (id 3) (at 146.304 84.328 0)
+      (effects (font (size 1.27 1.27)) hide)
+    )
+    (pin "1")
+  )
+  (symbol (lib_id "Device:C") (at 118.872 62.484 90) (unit 1)
+    (in_bom yes) (on_board yes) (fields_autoplaced)
+    (property "Reference" "Cpi21" (id 0) (at 118.872 54.61 90))
+    (property "Value" "C" (id 1) (at 118.872 57.15 90))
+    (property "Footprint" "Capacitor_SMD:C_0805_2012Metric_Pad1.18x1.45mm_HandSolder" (id 2) (at 122.682 61.5188 0)
+      (effects (font (size 1.27 1.27)) hide)
+    )
+    (property "Datasheet" "~" (id 3) (at 118.872 62.484 0)
+      (effects (font (size 1.27 1.27)) hide)
+    )
+    (pin "1")
+    (pin "2")
   )
 )

Commit message: PCB design done
Parts:
- Cpi1, Cpi11: value C -> 220p
- Cpi2, Cpi21: value C -> 33p
- Lpi1: value L -> 551.6nH
Changed lines of the file:
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@@
     (stroke (width 0) (type default) (color 0 0 0 0))
   )
-  (wire (pts (xy 98.552 73.66) (xy 102.87 73.66))
+  (wire (pts (xy 87.63 73.66) (xy 102.87 73.66))
     (stroke (width 0) (type default) (color 0 0 0 0))
   )
@@
     (stroke (width 0) (type default) (color 0 0 0 0))
   )
-  (hierarchical_label "RF_Antenna" (shape input) (at 98.552 73.66 180)
+  (hierarchical_label "RF_Antenna" (shape input) (at 87.63 73.66 180)
     (effects (font (size 1.27 1.27)) (justify right))
   )
@@
   (symbol (lib_id "Device:L") (at 129.286 80.264 0) (unit 1)
     (in_bom yes) (on_board yes) (fields_autoplaced)
-    (property "Reference" "Lpi1" (id 0) (at 131.572 78.9939 0)
+    (property "Reference" "Lpi1" (id 0) (at 130.81 78.9939 0)
       (effects (font (size 1.27 1.27)) (justify left))
     )
-    (property "Value" "L" (id 1) (at 131.572 81.5339 0)
+    (property "Value" "551.6nH" (id 1) (at 130.81 81.5339 0)
       (effects (font (size 1.27 1.27)) (justify left))
     )
@@
   (symbol (lib_id "Device:C") (at 118.872 73.66 90) (unit 1)
     (in_bom yes) (on_board yes) (fields_autoplaced)
-    (property "Reference" "Cpi2" (id 0) (at 118.872 66.294 90))
-    (property "Value" "C" (id 1) (at 118.872 68.834 90))
+    (property "Reference" "Cpi2" (id 0) (at 118.872 66.04 90))
+    (property "Value" "33p" (id 1) (at 118.872 68.58 90))
     (property "Footprint" "Capacitor_SMD:C_0805_2012Metric_Pad1.18x1.45mm_HandSolder" (id 2) (at 122.682 72.6948 0)
       (effects (font (size 1.27 1.27)) hide)
@@
       (effects (font (size 1.27 1.27)) (justify right))
     )
-    (property "Value" "C" (id 1) (at 96.52 81.026 0)
+    (property "Value" "220p" (id 1) (at 96.52 81.026 0)
       (effects (font (size 1.27 1.27)) (justify right))
     )
@@
       (effects (font (size 1.27 1.27)) (justify left))
     )
-    (property "Value" "C" (id 1) (at 113.03 81.2799 0)
+    (property "Value" "220p" (id 1) (at 113.03 81.2799 0)
       (effects (font (size 1.27 1.27)) (justify left))
     )
@@
     (in_bom yes) (on_board yes) (fields_autoplaced)
     (property "Reference" "Cpi21" (id 0) (at 118.872 54.61 90))
-    (property "Value" "C" (id 1) (at 118.872 57.15 90))
+    (property "Value" "33p" (id 1) (at 118.872 57.15 90))
     (property "Footprint" "Capacitor_SMD:C_0805_2012Metric_Pad1.18x1.45mm_HandSolder" (id 2) (at 122.682 61.5188 0)
       (effects (font (size 1.27 1.27)) hide)
